File: smdboard.sch (KiCad schematic (older format))
At the start: 40 parts, among them IC1 4017, IC2 555, J1 MICROUSB

Commit message: add first revision
Parts:
- removed D2: ~, symbol D
- added C10, C9: 100n, agg:0402-L, symbol C
- added C11: 10n, agg:0402-L, symbol C
- added C6, C7: 2µ2, agg:0603-L, symbol C
- added C8: 1µ, agg:0603-L, symbol C
- added D1, D10, D9: ~, agg:SOD-323, symbol D
- added D22, D23, D24, D25, D26, D27, D28, D29: LED, agg:0603-LED, symbol LED
- added IC3: STM32F091RxHx, agg:UFBGA-64, symbol STM32F091RxHx
- added P1: SWD_TC, agg:TC2030-NL, symbol SWD_TC
- added R100, R101, R102, R103, R92, R93, R94, R95, R96, R97, R98, R99: R, agg:0201-L, symbol R
- added R104, R105, R106, R107, R108, R109, R110, R111: 1k, agg:0402-L, symbol R
- added R14, R15, R16, R35, R36, R37, R56, R57, R58, R77, R78, R79: R, agg:0201, symbol R
- added R17, R18, R19, R38, R39, R40, R59, R60, R61, R80, R81, R82: R, agg:0402, symbol R
- added R20, R21, R22, R41, R42, R43, R62, R63, R64, R83, R84, R85: R, agg:0402-L, symbol R
- added R23, R24, R25, R44, R45, R46, R65, R66, R67, R86, R87, R88: R, agg:0603, symbol R
- added R26, R27, R28, R47, R48, R49, R68, R69, R70, R89, R90, R91: R, agg:0603-L, symbol R
- added R29, R30, R31, R50, R51, R52, R71, R72, R73, R74, R75, R76: R, agg:0805, symbol R
- added R32, R33, R34, R53, R54, R55: R, agg:1206, symbol R
- added TP1, TP2, TP3, TP4: TESTPAD, agg:WIREPAD, symbol TESTPAD
- added X1: MSOP-8, agg:MSOP-8, symbol PART
- added X3: LQFP-48, agg:LQFP-48, symbol PART
- added X4: QFN-48, agg:QFN-48-EP-ST, symbol PART
- added X9: LQFP-100, agg:LQFP-100, symbol PART
- C1, C2, C3, C4, C5, R1, R10, R11, R12, R13, R2, R3, R4, R5, R6, R7, R8, R9: footprint (none) -> agg:0805
- D11: renamed from D9; footprint (none) -> agg:0805-LED
- D12: renamed from D10; footprint (none) -> agg:0805-LED
- D13: renamed from D11; footprint (none) -> agg:0805-LED
- D14: renamed from D12; footprint (none) -> agg:0805-LED
- D15: renamed from D13; footprint (none) -> agg:0805-LED
- D16: renamed from D14; footprint (none) -> agg:0805-LED
- D17: renamed from D15; footprint (none) -> agg:0805-LED
- D18: renamed from D16; footprint (none) -> agg:0805-LED
- D19: renamed from D17; footprint (none) -> agg:0805-LED
- D2: renamed from D1; footprint (none) -> agg:SOD-323; Farnell (none) -> 1466524
- D20: renamed from D18; footprint (none) -> agg:0805-LED
- D21: renamed from D19; footprint (none) -> agg:0805-LED
- D3, D4, D5, D6, D7, D8: footprint (none) -> agg:SOD-323; Farnell (none) -> 1466524
- IC1: footprint agg:SOIC16 -> agg:SOIC-16
- IC2: footprint agg:SOIC8 -> agg:SOIC-8
- J1: footprint agg:USB3065 -> agg:MICROUSB_MOLEX_47589-0001; Farnell 2443111 -> 1568023
Connections:
- net GND: now also TP2.1 (TP)
- net VCC: now also TP1.1 (TP)
- net at D11.2, D21.2: now also D6.1; no longer IC1.1 (Q5)
- net at IC1.10 (Q4): now also D5.2; no longer D4.2
- net at IC1.11 (Q9): now also D10.2; no longer D8.2
- net at IC1.3 (Q0): now also D1.2; no longer D16.2
- net at IC1.4 (Q2): now also D3.2
- net at IC1.5 (Q6): now also D7.2; no longer D5.2
- net at D6.2: now also IC1.1 (Q5); no longer IC1.6 (Q7)
- net at IC1.7 (Q3): now also D4.2; no longer D3.2
- net at IC1.9 (Q8): now also D9.2; no longer D7.2
- net at D15.2, D17.2, D2.1: now also D10.1; no longer D8.1
- net at D12.2, D20.2, D5.1: now also D7.1; no longer D4.1
- net at D13.2, D19.2: now also D4.1, D8.1; no longer D3.1, D6.1
- net at D14.2, D18.2: now also D3.1, D9.1; no longer D7.1
- new net: D8.2, IC1.6 (Q7)
- new net: D1.1, D16.2
- new net: IC3.G8 (PB13), R111.1
- new net: IC3.H2 (PA1), R104.1
- new net: IC3.H3 (PA4), R105.1
- new net: IC3.H4 (PA7), R106.1
- new net: IC3.H5 (PC4), R107.1
- new net: IC3.H6 (PC5), R108.1
- new net: IC3.H7 (PB11), R109.1
- new net: IC3.H8 (PB12), R110.1
- new net: D25.2, R107.2
- new net: D26.2, R108.2
- new net: D27.2, R109.2
- new net: D28.2, R110.2
- new net: D29.2, R111.2
- new net: D23.2, R105.2
- new net: D22.2, R104.2
- new net: D24.2, R106.2
- new net DGND: C10.2, C11.2, C6.2, C7.2, C8.2, C9.2, D22.1, D23.1, D24.1, D25.1, D26.1, D27.1, D28.1, D29.1, IC3.B4 (BOOT0), IC3.C1 (PF0), IC3.C2 (VSS), IC3.C4 (PB5), IC3.D4 (VSS), IC3.D5 (VSS), IC3.D6 (VSS), IC3.D7 (PA8), IC3.D8 (PC9), IC3.F1 (VSSA), P1.5 (GND), TP4.1 (TP)
- new net NRST: IC3.E1 (NRST), P1.3 (~RST)
- new net PGND: R100.1, R100.2, R102.2, R103.1, R103.2, R15.2, R16.1, R16.2, R18.2, R19.1, R19.2, R21.2, R22.1, R22.2, R24.2, R25.1, R25.2, R27.2, R28.1, R28.2, R30.2, R31.1, R31.2, R33.2, R34.1, R34.2, R36.2, R37.1, R37.2, R39.2, R40.1, R40.2, R42.2, R43.1, R43.2, R45.2, R46.1, R46.2, R48.2, R49.1, R49.2, R51.2, R52.1, R52.2, R54.2, R55.1, R55.2, R57.2, R58.1, R58.2, R60.2, R61.1, R61.2, R63.2, R64.1, R64.2, R66.2, R67.1, R67.2, R69.2, R70.1, R70.2, R72.2, R73.1, R73.2, R75.2, R76.1, R76.2, R78.2, R79.1, R79.2, R81.2, R82.1, R82.2, R84.2, R85.1, R85.2, R87.2, R88.1, R88.2, R90.2, R91.1, R91.2, R93.2, R94.1, R94.2, R96.2, R97.1, R97.2, R99.2
- new net SWDCLK: IC3.A7 (PA14), P1.4 (SWDCLK)
- new net SWDIO: IC3.A8 (PA13), P1.2 (SWDIO)
- new net VDD: C10.1, C11.1, C6.1, C7.1, C8.1, C9.1, IC3.B2 (VBAT), IC3.B3 (PB8), IC3.C3 (PB7), IC3.D1 (PF1), IC3.D2 (VDD), IC3.D3 (PB6), IC3.E3 (PC0), IC3.E4 (VDD), IC3.E5 (VDD), IC3.E6 (VDDIO2), IC3.E7 (PC7), IC3.E8 (PC8), IC3.F3 (PA2), IC3.G1 (PC3), IC3.G2 (PA0), IC3.G3 (PA3), IC3.H1 (VDDA), P1.1 (VDD), TP3.1 (TP)
- no-connect marks 6 -> 123
Other:
- note added: "0201"
- note added: "0201-L"
- note added: "0402"
- note added: "0402-L"
- note added: "0603"
- note added: "0603-L"
- note added: "0805"
- note added: "1206"
- note added: "HARD MODE"
- note added: "SOLDER PRACTICE"

Commit message: Add Farnell order codes
Parts:
- C1, C2, C3, C4: Farnell (none) -> 2496944
- C10, C9: Farnell (none) -> 1759380
- C11: Farnell (none) -> 1758924
- C5: Farnell (none) -> 2497045
- C6, C7: Farnell (none) -> 2496923
- C8: Farnell (none) -> 2496916
- D11, D12, D13, D14, D15, D16, D17, D18, D19, D20, D21: Farnell (none) -> 5790840
- D22, D23, D24, D25, D26, D27, D28, D29: Farnell (none) -> 2290329
- R1, R2: Farnell (none) -> 2447551
- R10, R11, R12, R13, R3, R4, R5, R6, R7, R8, R9: Farnell (none) -> 2447552
- R104, R105, R106, R107, R108, R109, R110, R111: Farnell (none) -> 2447587
Changed lines of the file:
@@
 F 2 "agg:0805" H 3800 1500 60  0001 C CNN
 F 3 "" H 3800 1500 60  0000 C CNN
+F 4 "2447551" H 3800 1500 60  0001 C CNN "Farnell"
 	1    3800 1500
 	0    -1   -1   0
@@
 F 2 "agg:0805" H 3800 1700 60  0001 C CNN
 F 3 "" H 3800 1700 60  0000 C CNN
+F 4 "2447551" H 3800 1700 60  0001 C CNN "Farnell"
 	1    3800 1700
 	0    -1   -1   0
@@
 F 2 "agg:0805" H 3800 1900 60  0001 C CNN
 F 3 "" H 3800 1900 60  0000 C CNN
+F 4 "2497045" H 3800 1900 60  0001 C CNN "Farnell"
 	1    3800 1900
 	0    -1   -1   0
@@
 F 2 "agg:0805" H 4200 1350 60  0001 C CNN
 F 3 "" H 4200 1350 60  0000 C CNN
+F 4 "2496944" H 4200 1350 60  0001 C CNN "Farnell"
 	1    4200 1350
 	-1   0    0    1
@@
 F 2 "agg:0805" H 4200 1850 60  0001 C CNN
 F 3 "" H 4200 1850 60  0000 C CNN
+F 4 "2496944" H 4200 1850 60  0001 C CNN "Farnell"
 	1    4200 1850
 	0    1    1    0
@@
 F 2 "agg:0805" H 5300 950 60  0001 C CNN
 F 3 "" H 5300 950 60  0000 C CNN
+F 4 "2496944" H 5300 950 60  0001 C CNN "Farnell"
 	1    5300 950
 	-1   0    0    1
@@
 F 2 "agg:0805-LED" H 6550 2100 60  0001 C CNN
 F 3 "" H 6550 2100 60  0000 C CNN
+F 4 "5790840" H 6550 2100 60  0001 C CNN "Farnell"
 	1    6550 2100
 	0    -1   -1   0
@@
 F 2 "agg:0805" H 7050 2250 60  0001 C CNN
 F 3 "" H 7050 2250 60  0000 C CNN
+F 4 "2447552" H 7050 2250 60  0001 C CNN "Farnell"
 	1    7050 2250
 	0    -1   -1   0
@@
 F 2 "agg:0805" H 7300 2250 60  0001 C CNN
 F 3 "" H 7300 2250 60  0000 C CNN
+F 4 "2447552" H 7300 2250 60  0001 C CNN "Farnell"
 	1    7300 2250
 	0    -1   -1   0
@@
 F 2 "agg:0805" H 7550 2250 60  0001 C CNN
 F 3 "" H 7550 2250 60  0000 C CNN
+F 4 "2447552" H 7550 2250 60  0001 C CNN "Farnell"
 	1    7550 2250
 	0    -1   -1   0
@@
 F 2 "agg:0805" H 7800 2250 60  0001 C CNN
 F 3 "" H 7800 2250 60  0000 C CNN
+F 4 "2447552" H 7800 2250 60  0001 C CNN "Farnell"
 	1    7800 2250
 	0    -1   -1   0
@@
 F 2 "agg:0805" H 6800 2250 60  0001 C CNN
 F 3 "" H 6800 2250 60  0000 C CNN
+F 4 "2447552" H 6800 2250 60  0001 C CNN "Farnell"
 	1    6800 2250
 	0    -1   -1   0
@@
 F 2 "agg:0805" H 6550 2250 60  0001 C CNN
 F 3 "" H 6550 2250 60  0000 C CNN
+F 4 "2447552" H 6550 2250 60  0001 C CNN "Farnell"
 	1    6550 2250
 	0    -1   -1   0
@@
 F 2 "agg:0805" H 8050 2250 60  0001 C CNN
 F 3 "" H 8050 2250 60  0000 C CNN
+F 4 "2447552" H 8050 2250 60  0001 C CNN "Farnell"
 	1    8050 2250
 	0    -1   -1   0
@@
 F 2 "agg:0805" H 8300 2250 60  0001 C CNN
 F 3 "" H 8300 2250 60  0000 C CNN
+F 4 "2447552" H 8300 2250 60  0001 C CNN "Farnell"
 	1    8300 2250
 	0    -1   -1   0
@@
 F 2 "agg:0805" H 8550 2250 60  0001 C CNN
 F 3 "" H 8550 2250 60  0000 C CNN
+F 4 "2447552" H 8550 2250 60  0001 C CNN "Farnell"
 	1    8550 2250
 	0    -1   -1   0
@@
 F 2 "agg:0805" H 8800 2250 60  0001 C CNN
 F 3 "" H 8800 2250 60  0000 C CNN
+F 4 "2447552" H 8800 2250 60  0001 C CNN "Farnell"
 	1    8800 2250
 	0    -1   -1   0
@@
 F 2 "agg:0805" H 9050 2250 60  0001 C CNN
 F 3 "" H 9050 2250 60  0000 C CNN
+F 4 "2447552" H 9050 2250 60  0001 C CNN "Farnell"
 	1    9050 2250
 	0    -1   -1   0
@@
 F 2 "agg:0805-LED" H 6800 2100 60  0001 C CNN
 F 3 "" H 6800 2100 60  0000 C CNN
+F 4 "5790840" H 6800 2100 60  0001 C CNN "Farnell"
 	1    6800 2100
 	0    -1   -1   0
@@
 F 2 "agg:0805-LED" H 7050 2100 60  0001 C CNN
 F 3 "" H 7050 2100 60  0000 C CNN
+F 4 "5790840" H 7050 2100 60  0001 C CNN "Farnell"
 	1    7050 2100
 	0    -1   -1   0
@@
 F 2 "agg:0805-LED" H 7300 2100 60  0001 C CNN
 F 3 "" H 7300 2100 60  0000 C CNN
+F 4 "5790840" H 7300 2100 60  0001 C CNN "Farnell"
 	1    7300 2100
 	0    -1   -1   0
@@
 F 2 "agg:0805-LED" H 7550 2100 60  0001 C CNN
 F 3 "" H 7550 2100 60  0000 C CNN
+F 4 "5790840" H 7550 2100 60  0001 C CNN "Farnell"
 	1    7550 2100
 	0    -1   -1   0
@@
 F 2 "agg:0805-LED" H 7800 2100 60  0001 C CNN
 F 3 "" H 7800 2100 60  0000 C CNN
+F 4 "5790840" H 7800 2100 60  0001 C CNN "Farnell"
 	1    7800 2100
 	0    -1   -1   0
@@
 F 2 "agg:0805-LED" H 8050 2100 60  0001 C CNN
 F 3 "" H 8050 2100 60  0000 C CNN
+F 4 "5790840" H 8050 2100 60  0001 C CNN "Farnell"
 	1    8050 2100
 	0    -1   -1   0
@@
 F 2 "agg:0805-LED" H 8300 2100 60  0001 C CNN
 F 3 "" H 8300 2100 60  0000 C CNN
+F 4 "5790840" H 8300 2100 60  0001 C CNN "Farnell"
 	1    8300 2100
 	0    -1   -1   0
@@
 F 2 "agg:0805-LED" H 8550 2100 60  0001 C CNN
 F 3 "" H 8550 2100 60  0000 C CNN
+F 4 "5790840" H 8550 2100 60  0001 C CNN "Farnell"
 	1    8550 2100
 	0    -1   -1   0
@@
 F 2 "agg:0805-LED" H 8800 2100 60  0001 C CNN
 F 3 "" H 8800 2100 60  0000 C CNN
+F 4 "5790840" H 8800 2100 60  0001 C CNN "Farnell"
 	1    8800 2100
 	0    -1   -1   0
@@
 F 2 "agg:0805-LED" H 9050 2100 60  0001 C CNN
 F 3 "" H 9050 2100 60  0000 C CNN
+F 4 "5790840" H 9050 2100 60  0001 C CNN "Farnell"
 	1    9050 2100
 	0    -1   -1   0
@@
 F 2 "agg:0805" H 3500 1350 60  0001 C CNN
 F 3 "" H 3500 1350 60  0000 C CNN
+F 4 "2496944" H 3500 1350 60  0001 C CNN "Farnell"
 	1    3500 1350
 	-1   0    0    1
@@
 F 2 "agg:0402-L" H 1800 4750 60  0001 C CNN
 F 3 "" H 1800 4750 60  0000 C CNN
+F 4 "1759380" H 1800 4750 60  0001 C CNN "Farnell"
 	1    1800 4750
 	0    1    1    0
@@
 F 2 "agg:0402-L" H 1600 4750 60  0001 C CNN
 F 3 "" H 1600 4750 60  0000 C CNN
+F 4 "1759380" H 1600 4750 60  0001 C CNN "Farnell"
 	1    1600 4750
 	0    1    1    0
@@
 F 2 "agg:0603-L" H 1400 4750 60  0001 C CNN
 F 3 "" H 1400 4750 60  0000 C CNN
+F 4 "2496916" H 1400 4750 60  0001 C CNN "Farnell"
 	1    1400 4750
 	0    1    1    0
@@
 F 2 "agg:0603-L" H 1200 4750 60  0001 C CNN
 F 3 "" H 1200 4750 60  0000 C CNN
+F 4 "2496923" H 1200 4750 60  0001 C CNN "Farnell"
 	1    1200 4750
 	0    1    1    0
@@
 F 2 "agg:0603-L" H 1000 4750 60  0001 C CNN
 F 3 "" H 1000 4750 60  0000 C CNN
+F 4 "2496923" H 1000 4750 60  0001 C CNN "Farnell"
 	1    1000 4750
 	0    1    1    0
@@
 F 2 "agg:0402-L" H 2000 4750 60  0001 C CNN
 F 3 "" H 2000 4750 60  0000 C CNN
+F 4 "1758924" H 2000 4750 60  0001 C CNN "Farnell"
 	1    2000 4750
 	0    1    1    0
@@
 F 2 "agg:0402-L" H 2150 6500 60  0001 C CNN
 F 3 "" H 2150 6500 60  0000 C CNN
+F 4 "2447587" H 2150 6500 60  0001 C CNN "Farnell"
 	1    2150 6500
 	-1   0    0    -1
@@
 F 2 "agg:0603-LED" H 1900 6500 60  0001 C CNN
 F 3 "" H 1900 6500 60  0000 C CNN
+F 4 "2290329" H 1900 6500 60  0001 C CNN "Farnell"
 	1    1900 6500
 	1    0    0    1
@@
 F 2 "agg:0402-L" H 2150 6200 60  0001 C CNN
 F 3 "" H 2150 6200 60  0000 C CNN
+F 4 "2447587" H 2150 6200 60  0001 C CNN "Farnell"
 	1    2150 6200
 	-1   0    0    -1
@@
 F 2 "agg:0603-LED" H 1900 6200 60  0001 C CNN
 F 3 "" H 1900 6200 60  0000 C CNN
+F 4 "2290329" H 1900 6200 60  0001 C CNN "Farnell"
 	1    1900 6200
 	1    0    0    1
@@
 F 2 "agg:0402-L" H 2150 6800 60  0001 C CNN
 F 3 "" H 2150 6800 60  0000 C CNN
+F 4 "2447587" H 2150 6800 60  0001 C CNN "Farnell"
 	1    2150 6800
 	-1   0    0    -1
@@
 F 2 "agg:0603-LED" H 1900 6800 60  0001 C CNN
 F 3 "" H 1900 6800 60  0000 C CNN
+F 4 "2290329" H 1900 6800 60  0001 C CNN "Farnell"
 	1    1900 6800
 	1    0    0    1
@@
 F 2 "agg:0402-L" H 3350 4800 60  0001 C CNN
 F 3 "" H 3350 4800 60  0000 C CNN
+F 4 "2447587" H 3350 4800 60  0001 C CNN "Farnell"
 	1    3350 4800
 	1    0    0    -1
@@
 F 2 "agg:0603-LED" H 3600 4800 60  0001 C CNN
 F 3 "" H 3600 4800 60  0000 C CNN
+F 4 "2290329" H 3600 4800 60  0001 C CNN "Farnell"
 	1    3600 4800
 	-1   0    0    1
@@
 F 2 "agg:0402-L" H 3350 4900 60  0001 C CNN
 F 3 "" H 3350 4900 60  0000 C CNN
+F 4 "2447587" H 3350 4900 60  0001 C CNN "Farnell"
 	1    3350 4900
 	1    0    0    -1
@@
 F 2 "agg:0603-LED" H 3600 4900 60  0001 C CNN
 F 3 "" H 3600 4900 60  0000 C CNN
+F 4 "2290329" H 3600 4900 60  0001 C CNN "Farnell"
 	1    3600 4900
 	-1   0    0    1
@@
 F 2 "agg:0402-L" H 3350 7200 60  0001 C CNN
 F 3 "" H 3350 7200 60  0000 C CNN
+F 4 "2447587" H 3350 7200 60  0001 C CNN "Farnell"
 	1    3350 7200
 	1    0    0    -1
@@
 F 2 "agg:0603-LED" H 3600 7200 60  0001 C CNN
 F 3 "" H 3600 7200 60  0000 C CNN
+F 4 "2290329" H 3600 7200 60  0001 C CNN "Farnell"
 	1    3600 7200
 	-1   0    0    1
@@
 F 2 "agg:0402-L" H 3350 7300 60  0001 C CNN
 F 3 "" H 3350 7300 60  0000 C CNN
+F 4 "2447587" H 3350 7300 60  0001 C CNN "Farnell"
 	1    3350 7300
 	1    0    0    -1
@@
 F 2 "agg:0603-LED" H 3600 7300 60  0001 C CNN
 F 3 "" H 3600 7300 60  0000 C CNN
+F 4 "2290329" H 3600 7300 60  0001 C CNN "Farnell"
 	1    3600 7300
 	-1   0    0    1
@@
 F 2 "agg:0402-L" H 3350 7400 60  0001 C CNN
 F 3 "" H 3350 7400 60  0000 C CNN
+F 4 "2447587" H 3350 7400 60  0001 C CNN "Farnell"
 	1    3350 7400
 	1    0    0    -1
@@
 F 2 "agg:0603-LED" H 3600 7400 60  0001 C CNN
 F 3 "" H 3600 7400 60  0000 C CNN
+F 4 "2290329" H 3600 7400 60  0001 C CNN "Farnell"
 	1    3600 7400
 	-1   0    0    1
